Commit message: Changed environment config to scale up

File: TwoWheelBalance/src/TwoWheelBalance/assets/data/tw_balance.urdf (robot description, URDF)
Before this commit: robot balance_bot, 3 links, 2 joints
Links:
- link base_link: mass 1.0 -> 80.0; geometry collision box size=0.45 0.45 0.75; visual box size=0.45 0.45 0.75
- link left_wheel: mass 0.1 -> 5.0; geometry collision cylinder length=0.04 radius=0.3; visual cylinder length=0.04 radius=0.3
- link right_wheel: mass 0.1 -> 5.0; geometry collision cylinder length=0.04 radius=0.3; visual cylinder length=0.04 radius=0.3
Joints:
- joint left_wheel_joint: origin xyz=0 0.115 -0.05 rpy=0 0 0 -> xyz=0 0.305 -0.305 rpy=0 0 0
- joint right_wheel_joint: origin xyz=0 -0.115 -0.05 rpy=0 0 0 -> xyz=0 -0.305 -0.305 rpy=0 0 0

Commit message: Added bash env selector, added camera follow robot, camera changes, removed logs

File: TwoWheelBalance/src/TwoWheelBalance/assets/data/tw_balance.urdf (robot description, URDF)
Before this commit: robot balance_bot, 3 links, 2 joints
Links:
- link base_link: mass 80.0 -> 120.0
- link left_wheel: mass 5.0 -> 20.0
- link right_wheel: mass 5.0 -> 20.0

Commit message: Added proper rider mass, reduced robot mass + new inertia, changed critic to obtain mass

File: TwoWheelBalance/src/TwoWheelBalance/assets/data/tw_balance.urdf (robot description, URDF)
Before this commit: robot balance_bot, 3 links, 2 joints
Links:
- link base_link: mass 120.0 -> 55.0
- link left_wheel: mass 20.0 -> 5.0
- link right_wheel: mass 20.0 -> 5.0
